File: hardware/nextion_hmi/nextion_hmi.sch (KiCad schematic (older format))
At the start: 21 parts, among them J1 5VDC, J2 TX, J3 RJ45_Shielded, J4 RX, J5 GND, J6 UART, K1 X_Micro_SD_Card_Det, U1 STM32F051C8Tx, U2 W25Q32FVSS, U3 XPT2046TS

Commit message: schemos paruosimas
Parts:
- added C1, C5: C, symbol Device:C
- added J10: DIO, 1X01, symbol SparkFun-Connectors:CONN_01
- added J11: VDD, 1X01, symbol SparkFun-Connectors:CONN_01
- added J2: GND, 1X01, symbol SparkFun-Connectors:CONN_01
- added J8: ~RST, 1X01, symbol SparkFun-Connectors:CONN_01
- added J9: CLK, 1X01, symbol SparkFun-Connectors:CONN_01
- added Q1: BC817, symbol Transistor_BJT:BC817
- added R10, R11, R7, R9: 10k, symbol Device:R
- added R6: 3R9, symbol Device:R
- added R8: 2R7, symbol Device:R
- added U5: AMS1117-3.3, Package_TO_SOT_SMD:SOT-223-3_TabPin2, symbol Regulator_Linear:AMS1117-3.3
- renumbered C1 to C4, C4 to C7, J2 to J4, J4 to J5, J5 to J7, R6 to R1, R7 to R12, R1 to R13
Connections:
- wire segments 136 -> 179
Other:
- moved on the sheet: J3

Commit message: tarpinis kommitas
Parts:
- removed C1, C2, C3, C4, C5, C7: C, symbol Device:C
- removed J1: 5VDC, 1X01, symbol SparkFun-Connectors:CONN_01
- removed J10: DIO, 1X01, symbol SparkFun-Connectors:CONN_01
- removed J11: VDD, 1X01, symbol SparkFun-Connectors:CONN_01
- removed J2, J7: GND, 1X01, symbol SparkFun-Connectors:CONN_01
- removed J4: TX, 1X01, symbol SparkFun-Connectors:CONN_01
- removed J5: RX, 1X01, symbol SparkFun-Connectors:CONN_01
- removed J6: UART, symbol SparkFun-Connectors:CONN_04LOCK
- removed J8: ~RST, 1X01, symbol SparkFun-Connectors:CONN_01
- removed J9: CLK, 1X01, symbol SparkFun-Connectors:CONN_01
- removed K1: X_Micro_SD_Card_Det, symbol mech:X_Micro_SD_Card_Det
- removed Q1: BC817, symbol Transistor_BJT:BC817
- removed R1, R10, R11, R12, R13, R7, R9: 10k, symbol Device:R
- removed R2, R3, R4, R5: 4k7, symbol Device:R
- removed R6: 3R9, symbol Device:R
- removed R8: 2R7, symbol Device:R
- removed U1: STM32F051C8Tx, symbol ics:STM32F051C8Tx
- removed U2: W25Q32FVSS, symbol SparkFun-IC-Memory:W25Q32FVSS
- removed U3: XPT2046TS, symbol Driver_Display:XPT2046TS
- removed U5: AMS1117-3.3, Package_TO_SOT_SMD:SOT-223-3_TabPin2, symbol Regulator_Linear:AMS1117-3.3
- added C? (x2): 100nF, Capacitors_SMD:C_0805_HandSoldering, symbol Device:C
- added C? (x2): 100,0x16V, Capacitors_SMD:CP_Elec_8x6.5, symbol Device:CP
- added J1, J1A: UART, symbol SparkFun-Connectors:CONN_04SMD
- added U?: LM340-5.0-SMD, disc:TO-263-3_TabPin2, symbol disc:LM340-5.0-SMD
Connections:
- net labels removed: DATA_RX, DATA_TX, DAT_RX, DAT_TX, DISPLAY_LED, LCD_CS, LCD_DB0, LCD_DB1, LCD_DB10, LCD_DB11, LCD_DB12, LCD_DB13, LCD_DB14, LCD_DB15, LCD_DB2, LCD_DB3, LCD_DB4, LCD_DB5, LCD_DB6, LCD_DB7, LCD_DB8, LCD_DB9, LCD_RD, LCD_RS, LCD_RST, LCD_WR, SPI_MISO, SPI_MOSI, SPI_SCK, SWCLK, SWDIO, VDD, XN, XP, XPTCLK, XPTIN, XPTOUT, YN, YP, ~NRST, ~SDCS, ~SDDETECT, ~W25QCS, ~XPTCS, ~XPTREQ
- wire segments 179 -> 45
Other:
- moved on the sheet: J3
