File: hardware/nextion_hmi/uart_conv.sch (KiCad schematic (older format))
At the start: 18 parts, among them Q1 BC817, Q2 BC817, U4 LM340-5.0-SMD

Commit message: schemos paruosimas
Parts:
- renumbered C7 to C11
Changed lines of the file:
@@
 	1    0    0    1
 $EndComp
-Text HLabel 4100 4250 0    60   Input ~ 0
+Text HLabel 4100 4250 0    60   BiDi ~ 0
 DATA
 Connection ~ 4900 4850
@@
 Connection ~ 6850 2700
 $Comp
-L Device:C C7
+L Device:C C11
 U 1 1 5BFB2560
 P 5800 2900
-F 0 "C7" H 6000 2950 50  0000 C CNN
+F 0 "C11" H 6000 2950 50  0000 C CNN
 F 1 "100nF" H 6050 2850 50  0000 C CNN
 F 2 "Capacitors_SMD:C_0805_HandSoldering" H 5838 2750 50  0001 C CNN

Commit message: tarpinis kommitas
Parts:
- removed C11, C6: 100nF, Capacitors_SMD:C_0805_HandSoldering, symbol Device:C
- removed C5, C8: 100,0x16V, Capacitors_SMD:CP_Elec_8x6.5, symbol Device:CP
- removed D1, D2: BAS85, Diodes_SMD:D_MiniMELF_Handsoldering, symbol nextion_hmi-rescue:1N4148-
- removed U4: LM340-5.0-SMD, disc:TO-263-3_TabPin2, symbol disc:LM340-5.0-SMD
- renumbered C9 to C11, C10 to C12, D3 to D1, Q2 to Q3, R8 to R14, R9 to R15, R10 to R16, R11 to R17, R12 to R18, R13 to R19
Connections:
- net labels added: PF0, PF1, VDD
- net labels removed: 5VDC
- wire segments 52 -> 29
